File: MotorDriver/MotorDriver.sch (KiCad schematic (older format))
At the start: 17 parts, among them P1 CONN_01X04, P2 CONN_01X03, P4 CONN_01X02, U1 TB6593FNG

Commit message: finished motor driver layout and generated gerbers
Parts:
- C2, C4: footprint Capacitors_SMD:C_0805 -> Capacitors_SMD:C_1206_HandSoldering
- R1, R2, R3, R4: footprint Resistors_SMD:R_0805 -> Resistors_SMD:R_0805_HandSoldering
Changed lines of the file:
@@
 F 0 "C2" H 4970 3530 50  0000 L CNN
 F 1 "10u" H 5080 3370 50  0000 L CNN
-F 2 "Capacitors_SMD:C_0805" H 4970 3370 50  0001 C CNN
+F 2 "Capacitors_SMD:C_1206_HandSoldering" H 4970 3370 50  0001 C CNN
 F 3 "" H 4970 3370 50  0000 C CNN
 	1    4970 3370
@@
 F 0 "C4" H 6870 2870 50  0000 L CNN
 F 1 "10u" H 6660 2710 50  0000 L CNN
-F 2 "Capacitors_SMD:C_0805" H 6870 2710 50  0001 C CNN
+F 2 "Capacitors_SMD:C_1206_HandSoldering" H 6870 2710 50  0001 C CNN
 F 3 "" H 6870 2710 50  0000 C CNN
 	1    6870 2710
@@
 F 0 "R2" H 3780 4690 50  0000 L CNN
 F 1 "1K" H 3780 4630 50  0000 L CNN
-F 2 "Resistors_SMD:R_0805" H 3750 4670 50  0001 C CNN
+F 2 "Resistors_SMD:R_0805_HandSoldering" H 3750 4670 50  0001 C CNN
 F 3 "" H 3750 4670 50  0000 C CNN
 	1    3750 4670
@@
 F 0 "R4" H 4360 4690 50  0000 L CNN
 F 1 "1K" H 4360 4630 50  0000 L CNN
-F 2 "Resistors_SMD:R_0805" H 4330 4670 50  0001 C CNN
+F 2 "Resistors_SMD:R_0805_HandSoldering" H 4330 4670 50  0001 C CNN
 F 3 "" H 4330 4670 50  0000 C CNN
 	1    4330 4670
@@
 F 0 "R1" H 3760 3110 50  0000 L CNN
 F 1 "1K" H 3760 3050 50  0000 L CNN
-F 2 "Resistors_SMD:R_0805" H 3730 3090 50  0001 C CNN
+F 2 "Resistors_SMD:R_0805_HandSoldering" H 3730 3090 50  0001 C CNN
 F 3 "" H 3730 3090 50  0000 C CNN
 	1    3730 3090
@@
 F 0 "R3" H 4070 3110 50  0000 L CNN
 F 1 "1K" H 4070 3050 50  0000 L CNN
-F 2 "Resistors_SMD:R_0805" H 4040 3090 50  0001 C CNN
+F 2 "Resistors_SMD:R_0805_HandSoldering" H 4040 3090 50  0001 C CNN
 F 3 "" H 4040 3090 50  0000 C CNN
 	1    4040 3090
